Commit message: lf project

File: .gazebo/models/my_robot/model.urdf (robot description, URDF)
Before this commit: robot rrbot, 3 links, 2 joints
Links:
- removed link base_link
- removed link mid_link
- removed link top_link
- added link cas_wheel, mass 1; collision sphere radius=0.012; visual sphere radius=0.012
- added link chassis_back, mass 1; collision box size=0.025 0.05 0.005; visual box size=0.025 0.05 0.005
- added link chassis_front, mass 1; collision box size=0.06 0.016 0.005; visual box size=0.06 0.016 0.005
- added link wheel, mass 1; collision cylinder length=0.015 radius=0.012; visual cylinder length=0.015 radius=0.012
- added link wheel2, mass 1; collision cylinder length=0.015 radius=0.012; visual cylinder length=0.015 radius=0.012
Joints:
- removed joint joint_base_mid
- removed joint joint_mid_top
- added joint joint_front_back: type fixed, parent chassis_back, child chassis_front, origin xyz=0.042499999999999996 0 0 rpy=0 0 0
- added joint joint_left_wheel_back: type continuous, parent chassis_back, child wheel, origin xyz=0 0.0325 0 rpy=0 0 0, axis 0 1 0, limit lower=0.0 upper=0.0 effort=0.0 velocity=0.0
- added joint joint_right_wheel_back: type continuous, parent chassis_back, child wheel2, origin xyz=0 -0.0325 0 rpy=0 0 0, axis 0 1 0, limit lower=0.0 upper=0.0 effort=0.0 velocity=0.0

File: .gazebo/models/my_robot/model.xacro (robot description, xacro)
@@ -2,27 +2,108 @@
 <!-- Revolute-Revolute Manipulator -->
 <robot name="rrbot" xmlns:xacro="http://www.ros.org/wiki/xacro">
-  <!-- Constants for robot dimensions -->
-  <xacro:property name="width" value="0.1" />   <!-- Beams are square in length and width -->
-  <xacro:property name="height1" value="2" />   <!-- Link 1 -->
-  <xacro:property name="height2" value="1" />   <!-- Link 2 -->
-  <xacro:property name="height3" value="1" />   <!-- Link 3 -->
-  <xacro:property name="axle_offset" value="0.05" /> <!-- Space between joint and end of beam -->
-  <xacro:property name="damp" value="0.7" />    <!-- damping coefficient -->
-  <!-- Base Link -->
-  <link name="base_link">
+  <xacro:property name="x_ch_front" value="0.06" />   <!-- Beams are square in length and width -->
+  <xacro:property name="y_ch_front" value="0.016" />   <!-- Beams are square in length and width -->
+  <xacro:property name="z_ch_front" value="0.005" />   <!-- Beams are square in length and width -->
+  <xacro:property name="x_ch_back" value="0.025" />   <!-- Beams are square in length and width -->
+  <xacro:property name="y_ch_back" value="0.05" />   <!-- Beams are square in length and width -->
+  <xacro:property name="z_ch_back" value="0.005" />   <!-- Beams are square in length and width -->
+  <!-- WHEELS -->
+  <xacro:property name="wheel_rpy" value="1.55 0.0 0.0"/>
+  <xacro:property name="wheel_radius" value="0.012"/>
+  <xacro:property name="wheel_lenght" value="0.015"/>
+  <link name="cas_wheel">
+      <inertial>
+        <origin xyz="0 0 ${z_ch_front/2}" rpy="${wheel_rpy}"/>
+        <mass value="1"/>
+        <inertia
+          ixx="1.0" ixy="0.0" ixz="0.0"
+          iyy="1.0" iyz="0.0"
+          izz="1.0"/>
+      </inertial>
+      <visual>
+        <origin xyz="0 0 0 " rpy="${wheel_rpy}"/>
+        <geometry>
+          <sphere radius="${wheel_radius}" />
+        </geometry>
+        <material name="">
+          <color rgba="1.0 0.0 0.0 1.0"/>
+          <texture filename=""/>
+        </material>
+      </visual>
+      <collision>
+        <origin xyz="0 0 0 " rpy="${wheel_rpy}"/>
+        <geometry>
+          <sphere radius="${wheel_radius}"/>
+        </geometry>
+      </collision>
+    </link>
+  <link name="wheel">
+      <inertial>
+        <origin xyz="0 0 ${z_ch_front/2}" rpy="${wheel_rpy}"/>
+        <mass value="1"/>
+        <inertia
+          ixx="1.0" ixy="0.0" ixz="0.0"
+          iyy="1.0" iyz="0.0"
+          izz="1.0"/>
+      </inertial>
+      <visual>
+        <origin xyz="0 0 0 " rpy="${wheel_rpy}"/>
+        <geometry>
+          <cylinder radius="${wheel_radius}" length="${wheel_lenght}"/>
+        </geometry>
+        <material name="">
+          <color rgba="1.0 0.0 0.0 1.0"/>
+          <texture filename=""/>
+        </material>
+      </visual>
+      <collision>
+        <origin xyz="0 0 0 " rpy="${wheel_rpy}"/>
+        <geometry>
+          <cylinder radius="${wheel_radius}" length="${wheel_lenght}"/>
+        </geometry>
+      </collision>
+    </link>
+      <link name="wheel2">
+      <inertial>
+        <origin xyz="0 0 ${z_ch_front/2}" rpy="${wheel_rpy}"/>
+        <mass value="1"/>
+        <inertia
+          ixx="1.0" ixy="0.0" ixz="0.0"
+          iyy="1.0" iyz="0.0"
+          izz="1.0"/>
+      </inertial>
+      <visual>
+        <origin xyz="0 0 0 " rpy="${wheel_rpy}"/>
+        <geometry>
+          <cylinder radius="${wheel_radius}" length="${wheel_lenght}"/>
+        </geometry>
+        <material name="">
+          <color rgba="1.0 0.0 0.0 1.0"/>
+          <texture filename=""/>
+        </material>
+      </visual>
+      <collision>
+        <origin xyz="0 0 0 " rpy="${wheel_rpy}"/>
+        <geometry>
+          <cylinder radius="${wheel_radius}" length="${wheel_lenght}"/>
+        </geometry>
+      </collision>
+    </link>
+  <!-- Chassis front -->
+  <link name="chassis_front">
     <visual>
-      <origin xyz="0 0 ${height1/2}" rpy="0 0 0"/>
+      <origin xyz="0 0 ${z_ch_front/2}" rpy="0 0 0"/>
       <geometry>
-	<box size="${width} ${width} ${height1}"/>
+	<box size="${x_ch_front} ${y_ch_front} ${z_ch_front}"/>
       </geometry>
     </visual>
     <collision>
-      <origin xyz="0 0 ${height1/2}" rpy="0 0 0"/>
+      <origin xyz="0 0 ${z_ch_front/2}" rpy="0 0 0"/>
       <geometry>
-	<box size="${width} ${width} ${height1}"/>
+	<box size="${x_ch_front} ${y_ch_front} ${z_ch_front}"/>
       </geometry>
     </collision>
     <inertial>
-      <origin xyz="0 0 ${height1/2}" rpy="0 0 0"/>
+      <origin xyz="0 0 ${z_ch_front/2}" rpy="0 0 0"/>
       <mass value="1"/>
       <inertia
@@ -32,29 +113,20 @@
     </inertial>
   </link>
-  <!-- Joint between Base Link and Middle Link -->
-  <joint name="joint_base_mid" type="revolute">
-    <parent link="base_link"/>
-    <child link="mid_link"/>
-    <origin xyz="0 ${width} ${height1 - axle_offset}" rpy="0 0 0"/>
-    <axis xyz="0 1 0"/>
-    <dynamics damping="${damp}"/>
-    <limit effort="100.0" velocity="0.5" lower="-3.14" upper="3.14" />
-  </joint>
-  <!-- Middle Link -->
-  <link name="mid_link">
+  <!-- Chassis back -->
+  <link name="chassis_back">
     <visual>
-      <origin xyz="0 0 ${height2/2 - axle_offset}" rpy="0 0 0"/>
+      <origin xyz="0 0 ${z_ch_back/2}" rpy="0 0 0"/>
       <geometry>
-	<box size="${width} ${width} ${height2}"/>
+	<box size="${x_ch_back} ${y_ch_back} ${z_ch_back}"/>
       </geometry>
     </visual>
     <collision>
-      <origin xyz="0 0 ${height2/2 - axle_offset}" rpy="0 0 0"/>
+      <origin xyz="0 0 ${z_ch_back/2}" rpy="0 0 0"/>
       <geometry>
-	<box size="${width} ${width} ${height2}"/>
+	<box size="${x_ch_back} ${y_ch_back} ${z_ch_back}"/>
       </geometry>
     </collision>
     <inertial>
-      <origin xyz="0 0 ${height2/2 - axle_offset}" rpy="0 0 0"/>
+      <origin xyz="0 0 ${z_ch_back/2}" rpy="0 0 0"/>
       <mass value="1"/>
       <inertia
@@ -64,35 +136,33 @@
     </inertial>
   </link>
-  <!-- Joint between Middle Link and Top Link -->
-  <joint name="joint_mid_top" type="revolute">
-    <parent link="mid_link"/>
-    <child link="top_link"/>
-    <origin xyz="0 ${width} ${height2 - axle_offset*2}" rpy="0 0 0"/>
-    <axis xyz="0 1 0"/>
-    <dynamics damping="${damp}"/>
-    <limit effort="100.0" velocity="0.5" lower="-3.14" upper="3.14" />
+  <!-- Joint between both chassises -->
+  <joint name="joint_front_back" type="fixed">
+    <parent link="chassis_back"/>
+    <child link="chassis_front"/>
+    <origin xyz="${ (x_ch_front+x_ch_back) /2} 0 0" rpy="0 0 0"/>
   </joint>
-  <!-- Top Link -->
-  <link name="top_link">
-    <visual>
-      <origin xyz="0 0 ${height3/2 - axle_offset}" rpy="0 0 0"/>
-      <geometry>
-	<box size="${width} ${width} ${height3}"/>
-      </geometry>
-    </visual>
-    <collision>
-      <origin xyz="0 0 ${height3/2 - axle_offset}" rpy="0 0 0"/>
-      <geometry>
-	<box size="${width} ${width} ${height3}"/>
-      </geometry>
-    </collision>
-    <inertial>
-      <origin xyz="0 0 ${height3/2 - axle_offset}" rpy="0 0 0"/>
-      <mass value="1"/>
-      <inertia
-	  ixx="1.0" ixy="0.0" ixz="0.0"
-	  iyy="1.0" iyz="0.0"
-	  izz="1.0"/>
-    </inertial>
-  </link>
+  <!-- Joint between chassis back and wheel -->
+  <joint name="joint_left_wheel_back" type="continuous">
+    <parent link="chassis_back"/>
+    <child link="wheel"/>
+    <limit lower="0.0" upper="0.0" effort="0.0" velocity="0.0"/>
+    <origin xyz="0 ${y_ch_back/2+wheel_lenght/2} 0" rpy="0 0 0"/>
+    <axis xyz="0 1 0" rpy="0 0 0"/>
+  </joint>
+  <!-- Joint between chassis back and wheel -->
+  <joint name="joint_right_wheel_back" type="continuous">
+    <parent link="chassis_back"/>
+    <child link="wheel2"/>
+    <limit lower="0.0" upper="0.0" effort="0.0" velocity="0.0"/>
+    <origin xyz="0 ${-y_ch_back/2-wheel_lenght/2} 0" rpy="0 0 0"/>
+    <axis xyz="0 1 0" rpy="0 0 0"/>
+  </joint>
+  <!-- Joint between chassis back and wheel -->
+  <joint name="joint_cas_wheel_front" type="continuous">
+    <parent link="chassis_front"/>
+    <child link="cas_wheel"/>
+    <limit lower="0.0" upper="0.0" effort="0.0" velocity="0.0"/>
+    <origin xyz="0 ${-y_ch_back/2-wheel_lenght/2} 0" rpy="0 0 0"/>
+    <axis xyz="0 1 0" rpy="0 0 0"/>
+  </joint>
 </robot>

Commit message: lf project2

File: .gazebo/models/my_robot/model.urdf (robot description, URDF)
Before this commit: robot rrbot, 5 links, 3 joints
Links:
- added link chassis_mid, mass 0.3; collision box size=0.03 0.01 0.001; visual box size=0.03 0.01 0.001
- link cas_wheel: mass 1 -> 3; geometry collision sphere radius=0.005; visual sphere radius=0.005
- link chassis_back: mass 1 -> 2; geometry collision box size=0.025 0.04 0.001; visual box size=0.025 0.04 0.001
- link chassis_front: mass 1 -> 0.1; geometry collision box size=0.01 0.04 0.001; visual box size=0.01 0.04 0.001
- link wheel: mass 1 -> 3; geometry collision cylinder length=0.008 radius=0.012; visual cylinder length=0.008 radius=0.012
- link wheel2: mass 1 -> 3; geometry collision cylinder length=0.008 radius=0.012; visual cylinder length=0.008 radius=0.012
Joints:
- removed joint joint_front_back
- added joint joint_back_mid: type fixed, parent chassis_back, child chassis_mid, origin xyz=0.0275 0 0 rpy=0 0 0
- added joint joint_cas_wheel_mid: type continuous, parent chassis_mid, child cas_wheel, origin xyz=0 0 -0.005 rpy=0 0 0, axis 0 1 0, limit lower=0.0 upper=0.0 effort=0.0 velocity=0.0
- added joint joint_mid_front: type fixed, parent chassis_mid, child chassis_front, origin xyz=0.02 0 0 rpy=0 0 0
- joint joint_left_wheel_back: origin xyz=0 0.0325 0 rpy=0 0 0 -> xyz=0 0.024 0 rpy=0 0 0
- joint joint_right_wheel_back: origin xyz=0 -0.0325 0 rpy=0 0 0 -> xyz=0 -0.024 0 rpy=0 0 0

File: .gazebo/models/my_robot/model.xacro (robot description, xacro)
@@ -2,18 +2,22 @@
 <!-- Revolute-Revolute Manipulator -->
 <robot name="rrbot" xmlns:xacro="http://www.ros.org/wiki/xacro">
-  <xacro:property name="x_ch_front" value="0.06" />   <!-- Beams are square in length and width -->
-  <xacro:property name="y_ch_front" value="0.016" />   <!-- Beams are square in length and width -->
-  <xacro:property name="z_ch_front" value="0.005" />   <!-- Beams are square in length and width -->
+  <xacro:property name="x_ch_front" value="0.01" />   <!-- Beams are square in length and width -->
+  <xacro:property name="y_ch_front" value="0.04" />   <!-- Beams are square in length and width -->
+  <xacro:property name="z_ch_front" value="0.001" />   <!-- Beams are square in length and width -->
+  <xacro:property name="x_ch_mid" value="0.03" />   <!-- Beams are square in length and width -->
+  <xacro:property name="y_ch_mid" value="0.01" />   <!-- Beams are square in length and width -->
+  <xacro:property name="z_ch_mid" value="0.001" />   <!-- Beams are square in length and width -->
   <xacro:property name="x_ch_back" value="0.025" />   <!-- Beams are square in length and width -->
-  <xacro:property name="y_ch_back" value="0.05" />   <!-- Beams are square in length and width -->
-  <xacro:property name="z_ch_back" value="0.005" />   <!-- Beams are square in length and width -->
+  <xacro:property name="y_ch_back" value="0.04" />   <!-- Beams are square in length and width -->
+  <xacro:property name="z_ch_back" value="0.001" />   <!-- Beams are square in length and width -->
   <!-- WHEELS -->
   <xacro:property name="wheel_rpy" value="1.55 0.0 0.0"/>
   <xacro:property name="wheel_radius" value="0.012"/>
-  <xacro:property name="wheel_lenght" value="0.015"/>
+  <xacro:property name="wheel_lenght" value="0.008"/>
+  <xacro:property name="cas_wheel_radius" value="0.005"/>
   <link name="cas_wheel">
       <inertial>
-        <origin xyz="0 0 ${z_ch_front/2}" rpy="${wheel_rpy}"/>
-        <mass value="1"/>
+        <origin xyz="0 0 ${z_ch_mid/2}" rpy="${wheel_rpy}"/>
+        <mass value="3"/>
         <inertia
           ixx="1.0" ixy="0.0" ixz="0.0"
@@ -24,5 +28,5 @@
         <origin xyz="0 0 0 " rpy="${wheel_rpy}"/>
         <geometry>
-          <sphere radius="${wheel_radius}" />
+          <sphere radius="${cas_wheel_radius}" />
         </geometry>
         <material name="">
@@ -34,5 +38,5 @@
         <origin xyz="0 0 0 " rpy="${wheel_rpy}"/>
         <geometry>
-          <sphere radius="${wheel_radius}"/>
+          <sphere radius="${cas_wheel_radius}"/>
         </geometry>
       </collision>
@@ -40,6 +44,6 @@
   <link name="wheel">
       <inertial>
-        <origin xyz="0 0 ${z_ch_front/2}" rpy="${wheel_rpy}"/>
-        <mass value="1"/>
+        <origin xyz="0 0 ${z_ch_mid/2}" rpy="${wheel_rpy}"/>
+        <mass value="3"/>
         <inertia
           ixx="1.0" ixy="0.0" ixz="0.0"
@@ -66,6 +70,6 @@
       <link name="wheel2">
       <inertial>
-        <origin xyz="0 0 ${z_ch_front/2}" rpy="${wheel_rpy}"/>
-        <mass value="1"/>
+        <origin xyz="0 0 ${z_ch_mid/2}" rpy="${wheel_rpy}"/>
+        <mass value="3"/>
         <inertia
           ixx="1.0" ixy="0.0" ixz="0.0"
@@ -106,5 +110,28 @@
     <inertial>
       <origin xyz="0 0 ${z_ch_front/2}" rpy="0 0 0"/>
-      <mass value="1"/>
+      <mass value="0.1"/>
+      <inertia
+	  ixx="1.0" ixy="0.0" ixz="0.0"
+	  iyy="1.0" iyz="0.0"
+	  izz="1.0"/>
+    </inertial>
+  </link>
+  <!-- Chassis mid -->
+  <link name="chassis_mid">
+    <visual>
+      <origin xyz="0 0 ${z_ch_mid/2}" rpy="0 0 0"/>
+      <geometry>
+	<box size="${x_ch_mid} ${y_ch_mid} ${z_ch_mid}"/>
+      </geometry>
+    </visual>
+    <collision>
+      <origin xyz="0 0 ${z_ch_mid/2}" rpy="0 0 0"/>
+      <geometry>
+	<box size="${x_ch_mid} ${y_ch_mid} ${z_ch_mid}"/>
+      </geometry>
+    </collision>
+    <inertial>
+      <origin xyz="0 0 ${z_ch_mid/2}" rpy="0 0 0"/>
+      <mass value="0.3"/>
       <inertia
 	  ixx="1.0" ixy="0.0" ixz="0.0"
@@ -129,5 +156,5 @@
     <inertial>
       <origin xyz="0 0 ${z_ch_back/2}" rpy="0 0 0"/>
-      <mass value="1"/>
+      <mass value="2"/>
       <inertia
 	  ixx="1.0" ixy="0.0" ixz="0.0"
@@ -137,8 +164,14 @@
   </link>
   <!-- Joint between both chassises -->
-  <joint name="joint_front_back" type="fixed">
+  <joint name="joint_back_mid" type="fixed">
     <parent link="chassis_back"/>
+    <child link="chassis_mid"/>
+    <origin xyz="${ (x_ch_mid+x_ch_back) /2} 0 0" rpy="0 0 0"/>
+  </joint>
+   <!-- Joint between both chassises -->
+  <joint name="joint_mid_front" type="fixed">
+    <parent link="chassis_mid"/>
     <child link="chassis_front"/>
-    <origin xyz="${ (x_ch_front+x_ch_back) /2} 0 0" rpy="0 0 0"/>
+    <origin xyz="${ (x_ch_mid+x_ch_front) /2} 0 0" rpy="0 0 0"/>
   </joint>
   <!-- Joint between chassis back and wheel -->
@@ -159,9 +192,9 @@
   </joint>
   <!-- Joint between chassis back and wheel -->
-  <joint name="joint_cas_wheel_front" type="continuous">
-    <parent link="chassis_front"/>
+  <joint name="joint_cas_wheel_mid" type="continuous">
+    <parent link="chassis_mid"/>
     <child link="cas_wheel"/>
     <limit lower="0.0" upper="0.0" effort="0.0" velocity="0.0"/>
-    <origin xyz="0 ${-y_ch_back/2-wheel_lenght/2} 0" rpy="0 0 0"/>
+    <origin xyz="0 0 ${-cas_wheel_radius}" rpy="0 0 0"/>
     <axis xyz="0 1 0" rpy="0 0 0"/>
   </joint>

Commit message: clean

File: .gazebo/models/my_robot/model.urdf (robot description, URDF)
Before this commit: robot rrbot, 6 links, 5 joints
Links:
- link cas_wheel: mass 3 -> 10
- link wheel: mass 3 -> 30
- link wheel2: mass 3 -> 30

File: .gazebo/models/my_robot/model.xacro (robot description, xacro)
@@ -19,5 +19,5 @@
       <inertial>
         <origin xyz="0 0 ${z_ch_mid/2}" rpy="${wheel_rpy}"/>
-        <mass value="3"/>
+        <mass value="10"/>
         <inertia
           ixx="1.0" ixy="0.0" ixz="0.0"
@@ -45,5 +45,5 @@
       <inertial>
         <origin xyz="0 0 ${z_ch_mid/2}" rpy="${wheel_rpy}"/>
-        <mass value="3"/>
+        <mass value="30"/>
         <inertia
           ixx="1.0" ixy="0.0" ixz="0.0"
@@ -71,5 +71,5 @@
       <inertial>
         <origin xyz="0 0 ${z_ch_mid/2}" rpy="${wheel_rpy}"/>
-        <mass value="3"/>
+        <mass value="30"/>
         <inertia
           ixx="1.0" ixy="0.0" ixz="0.0"
@@ -199,3 +199,37 @@
     <axis xyz="0 1 0" rpy="0 0 0"/>
   </joint>
+      <gazebo>
+      <plugin name='control_p3d' filename='libgazebo_ros_p3d.so'>
+        <always_on>true</always_on>
+        <body_name>chassis_back</body_name>
+        <topic_name>odom</topic_name>
+        <frame_name>map</frame_name>
+        <update_rate>50</update_rate>
+      </plugin>
+      <plugin name='diff_drive' filename='libgazebo_ros_diff_drive.so'>
+        <ros>
+          <namespace>/lf</namespace>
+          <remapping>cmd_lf:=cmd_lf</remapping>
+          <remapping>odom:=odom_lf</remapping>
+        </ros>
+        <!-- wheels -->
+        <left_joint>left_wheel_joint</left_joint>
+        <right_joint>right_wheel_joint</right_joint>
+        <!-- kinematics -->
+        <wheel_separation>1.25</wheel_separation>
+        <wheel_diameter>0.6</wheel_diameter>
+        <!-- limits -->
+        <max_wheel_torque>20</max_wheel_torque>
+        <max_wheel_acceleration>1.0</max_wheel_acceleration>
+        <!-- output -->
+        <publish_odom>true</publish_odom>
+        <publish_odom_tf>true</publish_odom_tf>
+        <publish_wheel_tf>true</publish_wheel_tf>
+        <odom_publish>true</odom_publish>
+        <odometry_frame>map</odometry_frame>
+        <odom_frame_id>odom</odom_frame_id>
+        <robot_base_frame>chassis_back</robot_base_frame>
+        <always_on>true</always_on>
+      </plugin>
+      </gazebo>
 </robot>
